Commit message: status: finalizado

File: src/turtlebot4/turtlebot4_description/urdf/sensors/oakd.urdf.xacro (robot description, xacro)
@@ -17,5 +17,5 @@
     <parent link="${parent_link}"/>
     <child link="${base_frame}"/>
-    <origin xyz="0 0 0.20" rpy="0 -1.5707963 0"/>
+    <origin xyz="0 0 0.20" rpy="0 0 0"/>
   </joint>
   <link name="${base_frame}">
